File: trackball-sensor/trackball-sensor-3610.kicad_pcb (KiCad board)
At the start: 2 copper layers, 30 x 42.2 mm, 16 parts, among them J1 SM06B-SRSS-TB(LF)(SN), U1 TLV74318PDBVR, U2 PMW3610DM-SUDO

Commit message: Pin1 label
Other:
- board text added: "3610 REV0.3 - VINCENT FRANCO"
- board text added: "PIN1"
- board text removed: "REV0.2 - VINCENT FRANCO"
Changed lines of the file:
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@@
 		(tags "capacitor")
 		(property "Reference" "C1"
-			(at -0.15 1.525 0)
+			(at -0.05 -1.35 0)
 			(layer "B.SilkS")
 			(effects
@@
 	)
 	(gr_text "3.3\nSCLK\nMOTION\nMISO\nCS\nGND"
-		(at 140.58 94.73 0)
+		(at 141.625 94.45 0)
 		(layer "B.SilkS")
 		(effects
@@
 		)
 	)
-	(gr_text "REV0.2 - VINCENT FRANCO"
-		(at 115.6 110.8 270)
+	(gr_text "PIN1"
+		(at 132.625 104.8 180)
+		(layer "B.SilkS" knockout)
+		(effects
+			(font
+				(size 1.5 1.5)
+				(thickness 0.15)
+			)
+			(justify left bottom mirror)
+		)
+	)
+	(gr_text "3610 REV0.3 - VINCENT FRANCO"
+		(at 115.475 113.175 270)
 		(layer "B.SilkS" knockout)
 		(effects
@@
 	)
 	(via
-		(at 133.15 105.95)
+		(at 133.45 106.275)
 		(size 0.6)
 		(drill 0.3)
